Commit message: can run no fly

File: urdf/am_min.urdf (robot description, URDF)
Before this commit: robot aerial_manipulator, 4 links, 3 joints
Links:
- added link rotor_1, mass 0.05; collision cylinder length=0.02 radius=0.05; visual cylinder length=0.02 radius=0.05
- added link rotor_2, mass 0.05; collision cylinder length=0.02 radius=0.05; visual cylinder length=0.02 radius=0.05
- added link rotor_3, mass 0.05; collision cylinder length=0.02 radius=0.05; visual cylinder length=0.02 radius=0.05
- added link rotor_4, mass 0.05; collision cylinder length=0.02 radius=0.05; visual cylinder length=0.02 radius=0.05
Joints:
- added joint rotor_1_joint: type fixed, parent base_link, child rotor_1, origin xyz=0.15 0.15 0.06 rpy=0 0 0
- added joint rotor_2_joint: type fixed, parent base_link, child rotor_2, origin xyz=0.15 -0.15 0.06 rpy=0 0 0
- added joint rotor_3_joint: type fixed, parent base_link, child rotor_3, origin xyz=-0.15 0.15 0.06 rpy=0 0 0
- added joint rotor_4_joint: type fixed, parent base_link, child rotor_4, origin xyz=-0.15 -0.15 0.06 rpy=0 0 0

Commit message: can move arm

File: urdf/am_min.urdf (robot description, URDF)
Before this commit: robot aerial_manipulator, 8 links, 7 joints
Joints:
- joint arm_joint_2: origin xyz=0 0 0.1 rpy=0 0 0 -> xyz=0 0 -0.1 rpy=0 0 0

Commit message: modify am model

File: urdf/am_min.urdf (robot description, URDF)
Before this commit: robot aerial_manipulator, 8 links, 7 joints
Links:
- added link end_effector, mass 0.05; collision sphere radius=0.025; visual sphere radius=0.025
- added link support_left, mass 0.05; collision box size=0.35 0.01 0.3; visual box size=0.02 0.01 0.3
- added link support_right, mass 0.05; collision box size=0.35 0.01 0.3; visual box size=0.02 0.01 0.3
- link arm_link_1: geometry collision cylinder length=0.2 radius=0.01; visual cylinder length=0.2 radius=0.01
- link arm_link_2: geometry collision cylinder length=0.2 radius=0.01; visual cylinder length=0.2 radius=0.01
Joints:
- added joint end_effector_joint: type fixed, parent arm_link_2, child end_effector, origin xyz=0 0 -0.2 rpy=0 0 0
- added joint support_left_joint: type fixed, parent base_link, child support_left, origin xyz=0 0.2 0 rpy=0 0 0
- added joint support_right_joint: type fixed, parent base_link, child support_right, origin xyz=0 -0.2 0 rpy=0 0 0
- joint arm_joint_1: origin xyz=0 0 0 rpy=0 0 0 -> xyz=0 0 0 rpy=0 -0.3 0
- joint arm_joint_2: axis 0 0 1 -> 0 1 0; origin xyz=0 0 -0.1 rpy=0 0 0 -> xyz=0 0 -0.2 rpy=0 -1.27 0

Commit message: base mpc init

File: urdf/am_min.urdf (robot description, URDF)
Before this commit: robot aerial_manipulator, 11 links, 10 joints
Links:
- link arm_base_link: geometry visual cylinder length=0.05 radius=0.02
- link arm_link_1: geometry visual cylinder length=0.2 radius=0.01
- link arm_link_2: geometry visual cylinder length=0.2 radius=0.01
- link end_effector: geometry visual sphere radius=0.025
Joints:
- joint arm_joint_1: origin xyz=0 0 0 rpy=0 -0.3 0 -> xyz=0 0 0 rpy=0 0 0
- joint arm_joint_2: origin xyz=0 0 -0.2 rpy=0 -1.27 0 -> xyz=0 0 -0.2 rpy=0 -3.14 0

Commit message: two cost functions

File: urdf/am_min.urdf (robot description, URDF)
Before this commit: robot aerial_manipulator, 11 links, 10 joints
Joints:
- joint arm_joint_2: origin xyz=0 0 -0.2 rpy=0 -3.14 0 -> xyz=0 0 -0.2 rpy=0 -1.57 0
